Commit message: modified:   calculator/src/function.cpp 	modified:   manager/src/manager.cpp 	modified:   robot_control/src/control.cpp 	modified:   robot_description/urdf/robot.urdf 	modified:   robot_description/urdf/robot_0.urdf 	modified:   robot_description/urdf/robot_1.urdf 	new file:   robot_description/urdf/robot_2.urdf

File: robot_description/urdf/robot_0.urdf (robot description, URDF)
Before this commit: robot robot_0, 7 links, 6 joints
Links:
- removed link caster_link
- added link after_caster_link, mass 0.02; collision sphere radius=0.016; visual sphere radius=0.016
- added link front_caster_link, mass 0.02; collision sphere radius=0.016; visual sphere radius=0.016
Joints:
- removed joint caster_joint
- added joint after_caster_joint: type fixed, parent base_link, child after_caster_link, origin xyz=-0.06 0.0 -0.076, axis 0 1 0
- added joint front_caster_joint: type fixed, parent base_link, child front_caster_link, origin xyz=0.06 0.0 -0.076, axis 0 1 0

File: robot_description/urdf/robot_2.urdf (robot description, URDF)
Before this commit: robot car_robot, 8 links, 7 joints
Links:
- removed link after_caster_link
- removed link front_caster_link
- added link caster_link, mass 0.02; collision sphere radius=0.016; visual sphere radius=0.016
Joints:
- removed joint after_caster_joint
- removed joint front_caster_joint
- added joint caster_joint: type fixed, parent base_link, child caster_link, origin xyz=0.06 0.0 -0.076, axis 0 1 0
