Commit message: modified:   calculator/include/calculator/common.hpp 	modified:   calculator/include/calculator/function.hpp 	modified:   calculator/include/calculator/marco.hpp 	modified:   calculator/src/function.cpp 	modified:   manager/CMakeLists.txt 	modified:   manager/include/manager/manager.hpp 	modified:   manager/include/manager/manager_interfaces.hpp 	modified:   manager/src/manager.cpp 	modified:   robot_control/CMakeLists.txt 	modified:   robot_control/include/robot_control/control.hpp 	new file:   robot_control/include/robot_control/joint_state.hpp 	modified:   robot_control/include/robot_control/robot_interfaces.hpp 	modified:   robot_control/src/control.cpp 	new file:   robot_control/src/joint_state.cpp 	new file:   robot_description/cartographer_config/robot_config.lua 	new file:   robot_description/launch/enviroment.launch.py 	modified:   robot_description/launch/robot.launch.py 	modified:   robot_description/setup.py 	renamed:    robot_description/urdf/robot.urdf -> robot_description/urdf/robot.urdf.xacro 	deleted:    robot_description/urdf/robot_0.urdf 	deleted:    robot_description/urdf/robot_1.urdf 	deleted:    robot_description/urdf/robot_2.urdf

File: robot_description/urdf/robot.urdf.xacro (robot description, xacro)
@@ -1,4 +1,5 @@
 <?xml version="1.0"?>
-<robot name="car_robot">
+<robot xmlns:xacro="http://www.ros.org/wiki/xacro" name="$(arg robot_name)">
+  <xacro:arg name="robot_name" default="robot"/>
   <!-- Robot Footprint -->
   <link name="base_footprint"/>
@@ -11,11 +12,11 @@
   <!-- base link -->
   <link name="base_link">
-  	<visual>
+    <visual>
       <origin xyz="0 0 0.0" rpy="0 0 0"/>
       <geometry>
-		<cylinder length="0.12" radius="0.10"/>
+    <cylinder length="0.12" radius="0.10"/>
       </geometry>
       <material name="blue">
-      	<color rgba="0.1 0.1 1.0 0.5" />
+        <color rgba="0.1 0.1 1.0 0.5" />
       </material>
     </visual>
@@ -23,8 +24,8 @@
       <origin xyz="0 0 0.0" rpy="0 0 0"/>
       <geometry>
-		<cylinder length="0.12" radius="0.10"/>
+    <cylinder length="0.12" radius="0.10"/>
       </geometry>
       <material name="blue">
-      	<color rgba="0.1 0.1 1.0 0.5" />
+        <color rgba="0.1 0.1 1.0 0.5" />
       </material>
     </collision>
@@ -67,8 +68,8 @@
   <!-- imu link -->
   <link name="imu_link">
-  	<visual>
+    <visual>
       <origin xyz="0 0 0.0" rpy="0 0 0"/>
       <geometry>
-		    <box size="0.02 0.02 0.02"/>
+        <box size="0.02 0.02 0.02"/>
       </geometry>
     </visual>
@@ -76,5 +77,5 @@
       <origin xyz="0 0 0.0" rpy="0 0 0"/>
       <geometry>
-		    <box size="0.02 0.02 0.02"/>
+        <box size="0.02 0.02 0.02"/>
       </geometry>
     </collision>
@@ -115,5 +116,5 @@
         </inertial>
   </link>
-  <!-- right_wheellink -->
+  <!-- right_wheel link -->
   <link name="right_wheel_link">
       <visual>
@@ -237,7 +238,7 @@
   </gazebo>
   <gazebo>
-    <plugin name='diff_drive' filename='libgazebo_ros_diff_drive.so'>
+    <plugin name="diff_drive" filename="libgazebo_ros_diff_drive.so">
           <ros>
-            <namespace>/</namespace>
+            <namespace>/$(arg robot_name)</namespace>
             <remapping>cmd_vel:=cmd_vel</remapping>
             <remapping>odom:=odom</remapping>
@@ -265,5 +266,5 @@
     <plugin filename="libgazebo_ros_imu_sensor.so" name="imu_plugin">
         <ros>
-          <namespace>/</namespace>
+          <namespace>/$(arg robot_name)</namespace>
           <remapping>~/out:=imu</remapping>
         </ros>
@@ -357,4 +358,5 @@
       <plugin name="laserscan" filename="libgazebo_ros_ray_sensor.so">
         <ros>
+          <namespace>/$(arg robot_name)</namespace>
           <remapping>~/out:=scan</remapping>
         </ros>

Commit message: modified:   calculator/include/calculator/marco.hpp 	modified:   robot_control/CMakeLists.txt 	modified:   robot_control/include/robot_control/control.hpp 	deleted:    robot_control/include/robot_control/joint_state.hpp 	modified:   robot_control/include/robot_control/robot_interfaces.hpp 	modified:   robot_control/src/control.cpp 	deleted:    robot_control/src/joint_state.cpp 	modified:   robot_description/launch/robot.launch.py 	modified:   robot_description/urdf/robot.urdf.xacro

File: robot_description/urdf/robot.urdf.xacro (robot description, xacro)
@@ -1,7 +1,32 @@
-<?xml version="1.0"?>
+<?xml version="1.0" encoding="utf-8"?>
 <robot xmlns:xacro="http://www.ros.org/wiki/xacro" name="$(arg robot_name)">
   <xacro:arg name="robot_name" default="robot"/>
   <!-- Robot Footprint -->
   <link name="base_footprint"/>
+  <!-- base link -->
+  <link name="base_link">
+    <visual>
+      <origin xyz="0 0 0.0" rpy="0 0 0"/>
+      <geometry>
+        <cylinder length="0.12" radius="0.10"/>
+      </geometry>
+      <material name="blue">
+        <color rgba="0.1 0.1 1.0 0.5"/>
+      </material>
+    </visual>
+    <collision>
+      <origin xyz="0 0 0.0" rpy="0 0 0"/>
+      <geometry>
+        <cylinder length="0.12" radius="0.10"/>
+      </geometry>
+      <material name="blue">
+        <color rgba="0.1 0.1 1.0 0.5"/>
+      </material>
+    </collision>
+    <inertial>
+      <mass value="0.2"/>
+      <inertia ixx="0.0122666" ixy="0" ixz="0" iyy="0.0122666" iyz="0" izz="0.02"/>
+    </inertial>
+  </link>
   <!-- base joint -->
   <joint name="base_joint" type="fixed">
@@ -10,29 +35,4 @@
     <origin xyz="0.0 0.0 0.076" rpy="0 0 0"/>
   </joint>
-  <!-- base link -->
-  <link name="base_link">
-    <visual>
-      <origin xyz="0 0 0.0" rpy="0 0 0"/>
-      <geometry>
-    <cylinder length="0.12" radius="0.10"/>
-      </geometry>
-      <material name="blue">
-        <color rgba="0.1 0.1 1.0 0.5" />
-      </material>
-    </visual>
-    <collision>
-      <origin xyz="0 0 0.0" rpy="0 0 0"/>
-      <geometry>
-    <cylinder length="0.12" radius="0.10"/>
-      </geometry>
-      <material name="blue">
-        <color rgba="0.1 0.1 1.0 0.5" />
-      </material>
-    </collision>
-    <inertial>
-      <mass value="0.2"/>
-      <inertia ixx="0.0122666" ixy="0" ixz="0" iyy="0.0122666" iyz="0" izz="0.02"/>
-    </inertial>
-  </link>
   <!-- laser link -->
   <link name="laser_link">
@@ -43,5 +43,5 @@
       </geometry>
       <material name="black">
-        <color rgba="0.0 0.0 0.0 0.5" />
+        <color rgba="0.0 0.0 0.0 0.5"/>
       </material>
     </visual>
@@ -52,9 +52,9 @@
       </geometry>
       <material name="black">
-        <color rgba="0.0 0.0 0.0 0.5" />
-      </material>
-    </collision>
-    <inertial>
-    <mass value="0.1"/>
+        <color rgba="0.0 0.0 0.0 0.5"/>
+      </material>
+    </collision>
+    <inertial>
+      <mass value="0.1"/>
       <inertia ixx="0.000190416666667" ixy="0" ixz="0" iyy="0.0001904" iyz="0" izz="0.00036"/>
     </inertial>
@@ -62,7 +62,7 @@
   <!-- laser joint -->
   <joint name="laser_joint" type="fixed">
-      <parent link="base_link" />
-      <child link="laser_link" />
-      <origin xyz="0 0 0.075" />
+    <parent link="base_link"/>
+    <child link="laser_link"/>
+    <origin xyz="0 0 0.075"/>
   </joint>
   <!-- imu link -->
@@ -82,98 +82,98 @@
     <inertial>
       <mass value="0.1"/>
-        <inertia ixx="0.000190416666667" ixy="0" ixz="0" iyy="0.0001904" iyz="0" izz="0.00036"/>
-      </inertial>
+      <inertia ixx="0.000190416666667" ixy="0" ixz="0" iyy="0.0001904" iyz="0" izz="0.00036"/>
+    </inertial>
   </link>
   <!-- imu joint -->
   <joint name="imu_joint" type="fixed">
-      <parent link="base_link" />
-      <child link="imu_link" />
-      <origin xyz="0 0 0.02" />
+    <parent link="base_link"/>
+    <child link="imu_link"/>
+    <origin xyz="0 0 0.02"/>
   </joint>
   <!-- left_wheel link -->
   <link name="left_wheel_link">
-      <visual>
-        <origin xyz="0 0 0" rpy="1.57079 0 0"/>
-        <geometry>
-          <cylinder length="0.04" radius="0.032"/>
-        </geometry>
-          <material name="black">
-            <color rgba="0.0 0.0 0.0 0.5" />
-          </material>
-      </visual>
-      <collision>
-        <origin xyz="0 0 0" rpy="1.57079 0 0"/>
-        <geometry>
-          <cylinder length="0.04" radius="0.032"/>
-        </geometry>
-          <material name="black">
-            <color rgba="0.0 0.0 0.0 0.5" />
-          </material>
-      </collision>
-      <inertial>
-        <mass value="0.2"/>
-          <inertia ixx="0.000190416666667" ixy="0" ixz="0" iyy="0.0001904" iyz="0" izz="0.00036"/>
-        </inertial>
-  </link>
+    <visual>
+      <origin xyz="0 0 0" rpy="1.57079 0 0"/>
+      <geometry>
+        <cylinder length="0.04" radius="0.032"/>
+      </geometry>
+      <material name="black">
+        <color rgba="0.0 0.0 0.0 0.5"/>
+      </material>
+    </visual>
+    <collision>
+      <origin xyz="0 0 0" rpy="1.57079 0 0"/>
+      <geometry>
+        <cylinder length="0.04" radius="0.032"/>
+      </geometry>
+      <material name="black">
+        <color rgba="0.0 0.0 0.0 0.5"/>
+      </material>
+    </collision>
+    <inertial>
+      <mass value="0.2"/>
+      <inertia ixx="0.000190416666667" ixy="0" ixz="0" iyy="0.0001904" iyz="0" izz="0.00036"/>
+    </inertial>
+  </link>
+  <!-- left_wheel joint -->
+  <joint name="left_wheel_joint" type="continuous">
+    <parent link="base_link"/>
+    <child link="left_wheel_link"/>
+    <origin xyz="-0.02 0.10 -0.06"/>
+    <axis xyz="0 1 0"/>
+  </joint>
   <!-- right_wheel link -->
   <link name="right_wheel_link">
-      <visual>
-        <origin xyz="0 0 0" rpy="1.57079 0 0"/>
-        <geometry>
-          <cylinder length="0.04" radius="0.032"/>
-        </geometry>
-          <material name="black">
-            <color rgba="0.0 0.0 0.0 0.5" />
-          </material>
-      </visual>
-      <collision>
-        <origin xyz="0 0 0" rpy="1.57079 0 0"/>
-        <geometry>
-          <cylinder length="0.04" radius="0.032"/>
-        </geometry>
-          <material name="black">
-            <color rgba="0.0 0.0 0.0 0.5" />
-          </material>
-      </collision>
-      <inertial>
+    <visual>
+      <origin xyz="0 0 0" rpy="1.57079 0 0"/>
+      <geometry>
+        <cylinder length="0.04" radius="0.032"/>
+      </geometry>
+      <material name="black">
+        <color rgba="0.0 0.0 0.0 0.5"/>
+      </material>
+    </visual>
+    <collision>
+      <origin xyz="0 0 0" rpy="1.57079 0 0"/>
+      <geometry>
+        <cylinder length="0.04" radius="0.032"/>
+      </geometry>
+      <material name="black">
+        <color rgba="0.0 0.0 0.0 0.5"/>
+      </material>
+    </collision>
+    <inertial>
       <mass value="0.2"/>
       <inertia ixx="0.000190416666667" ixy="0" ixz="0" iyy="0.0001904" iyz="0" izz="0.00036"/>
     </inertial>
   </link>
-  <!-- left_wheel joint -->
-  <joint name="left_wheel_joint" type="continuous">
-      <parent link="base_link" />
-      <child link="left_wheel_link" />
-      <origin xyz="-0.02 0.10 -0.06" />
-      <axis xyz="0 1 0" />
-  </joint>
   <!-- right_wheel joint -->
   <joint name="right_wheel_joint" type="continuous">
-      <parent link="base_link" />
-      <child link="right_wheel_link" />
-      <origin xyz="-0.02 -0.10 -0.06" />
-      <axis xyz="0 1 0" />
+    <parent link="base_link"/>
+    <child link="right_wheel_link"/>
+    <origin xyz="-0.02 -0.10 -0.06"/>
+    <axis xyz="0 1 0"/>
   </joint>
   <!-- fornt caster link -->
   <link name="front_caster_link">
-      <visual>
-        <origin xyz="0 0 0" rpy="1.57079 0 0"/>
-        <geometry>
-            <sphere radius="0.016"/>
-        </geometry>
-          <material name="black">
-            <color rgba="0.0 0.0 0.0 0.5" />
-          </material>
-      </visual>
-      <collision>
-        <origin xyz="0 0 0" rpy="1.57079 0 0"/>
-        <geometry>
-            <sphere radius="0.016"/>
-        </geometry>
-          <material name="black">
-            <color rgba="0.0 0.0 0.0 0.5" />
-          </material>
-      </collision>
-      <inertial>
+    <visual>
+      <origin xyz="0 0 0" rpy="1.57079 0 0"/>
+      <geometry>
+        <sphere radius="0.016"/>
+      </geometry>
+      <material name="black">
+        <color rgba="0.0 0.0 0.0 0.5"/>
+      </material>
+    </visual>
+    <collision>
+      <origin xyz="0 0 0" rpy="1.57079 0 0"/>
+      <geometry>
+        <sphere radius="0.016"/>
+      </geometry>
+      <material name="black">
+        <color rgba="0.0 0.0 0.0 0.5"/>
+      </material>
+    </collision>
+    <inertial>
       <mass value="0.02"/>
       <inertia ixx="0.000190416666667" ixy="0" ixz="0" iyy="0.0001904" iyz="0" izz="0.00036"/>
@@ -182,8 +182,8 @@
   <!-- front caster joint -->
   <joint name="front_caster_joint" type="fixed">
-      <parent link="base_link" />
-      <child link="front_caster_link" />
-      <origin xyz="0.06 0.0 -0.076" />
-      <axis xyz="0 1 0" />
+    <parent link="base_link"/>
+    <child link="front_caster_link"/>
+    <origin xyz="0.06 0.0 -0.076"/>
+    <axis xyz="0 1 0"/>
   </joint>
   <gazebo reference="front_caster_link">
@@ -193,28 +193,28 @@
     <mu1 value="0.0"/>
     <mu2 value="0.0"/>
-    <kp value="1000000.0" />
-    <kd value="10.0" />
-  </gazebo>
-<!-- after caster link -->
+    <kp value="1000000.0"/>
+    <kd value="10.0"/>
+  </gazebo>
+  <!-- after caster link -->
   <link name="after_caster_link">
-      <visual>
-        <origin xyz="0 0 0" rpy="1.57079 0 0"/>
-        <geometry>
-            <sphere radius="0.016"/>
-        </geometry>
-          <material name="black">
-            <color rgba="0.0 0.0 0.0 0.5" />
-          </material>
-      </visual>
-      <collision>
-        <origin xyz="0 0 0" rpy="1.57079 0 0"/>
-        <geometry>
-            <sphere radius="0.016"/>
-        </geometry>
-          <material name="black">
-            <color rgba="0.0 0.0 0.0 0.5" />
-          </material>
-      </collision>
-      <inertial>
+    <visual>
+      <origin xyz="0 0 0" rpy="1.57079 0 0"/>
+      <geometry>
+        <sphere radius="0.016"/>
+      </geometry>
+      <material name="black">
+        <color rgba="0.0 0.0 0.0 0.5"/>
+      </material>
+    </visual>
+    <collision>
+      <origin xyz="0 0 0" rpy="1.57079 0 0"/>
+      <geometry>
+        <sphere radius="0.016"/>
+      </geometry>
+      <material name="black">
+        <color rgba="0.0 0.0 0.0 0.5"/>
+      </material>
+    </collision>
+    <inertial>
       <mass value="0.02"/>
       <inertia ixx="0.000190416666667" ixy="0" ixz="0" iyy="0.0001904" iyz="0" izz="0.00036"/>
@@ -223,8 +223,8 @@
   <!-- after caster joint -->
   <joint name="after_caster_joint" type="fixed">
-      <parent link="base_link" />
-      <child link="after_caster_link" />
-      <origin xyz="-0.06 0.0 -0.076" />
-      <axis xyz="0 1 0" />
+    <parent link="base_link"/>
+    <child link="after_caster_link"/>
+    <origin xyz="-0.06 0.0 -0.076"/>
+    <axis xyz="0 1 0"/>
   </joint>
   <gazebo reference="after_caster_link">
@@ -234,35 +234,35 @@
     <mu1 value="0.0"/>
     <mu2 value="0.0"/>
-    <kp value="1000000.0" />
-    <kd value="10.0" />
+    <kp value="1000000.0"/>
+    <kd value="10.0"/>
   </gazebo>
   <gazebo>
     <plugin name="diff_drive" filename="libgazebo_ros_diff_drive.so">
-          <ros>
-            <namespace>/$(arg robot_name)</namespace>
-            <remapping>cmd_vel:=cmd_vel</remapping>
-            <remapping>odom:=odom</remapping>
-          </ros>
-          <update_rate>30</update_rate>
-          <!-- wheels -->
-          <left_joint>left_wheel_joint</left_joint>
-          <right_joint>right_wheel_joint</right_joint>
-          <!-- kinematics -->
-          <wheel_separation>0.2</wheel_separation>
-          <wheel_diameter>0.065</wheel_diameter>
-          <!-- limits -->
-          <max_wheel_torque>20</max_wheel_torque>
-          <max_wheel_acceleration>1.0</max_wheel_acceleration>
-          <!-- output -->
-          <publish_odom>true</publish_odom>
-          <publish_odom_tf>true</publish_odom_tf>
-          <publish_wheel_tf>true</publish_wheel_tf>
-          <odometry_frame>odom</odometry_frame>
-          <robot_base_frame>base_footprint</robot_base_frame>
+      <ros>
+        <namespace>/$(arg robot_name)</namespace>
+        <remapping>cmd_vel:=cmd_vel</remapping>
+        <remapping>odom:=odom</remapping>
+      </ros>
+      <update_rate>30</update_rate>
+      <!-- wheels -->
+      <left_joint>left_wheel_joint</left_joint>
+      <right_joint>right_wheel_joint</right_joint>
+      <!-- kinematics -->
+      <wheel_separation>0.2</wheel_separation>
+      <wheel_diameter>0.065</wheel_diameter>
+      <!-- limits -->
+      <max_wheel_torque>20</max_wheel_torque>
+      <max_wheel_acceleration>1.0</max_wheel_acceleration>
+      <!-- output -->
+      <publish_odom>true</publish_odom>
+      <publish_odom_tf>true</publish_odom_tf>
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