Commit message: new file:   manager/include/manager/global_map.hpp 	new file:   manager/src/global_map.cpp 	modified:   manager/src/manager.cpp 	modified:   robot_control/src/control.cpp 	new file:   robot_description/cartographer_config/cartographer_config.py 	modified:   robot_description/cartographer_config/robot_config.lua 	renamed:    robot_description/launch/urdf.launch.py -> robot_description/launch/config.launch.py 	modified:   robot_description/launch/enviroment.launch.py 	modified:   robot_description/launch/robot.launch.py 	modified:   robot_description/urdf/robot.urdf.xacro

File: robot_description/urdf/robot.urdf.xacro (robot description, xacro)
@@ -3,7 +3,7 @@
   <xacro:arg name="robot_name" default="robot"/>
   <!-- Robot Footprint -->
-  <link name="base_footprint"/>
+  <link name="$(arg robot_name)_base_footprint"/>
   <!-- base link -->
-  <link name="base_link">
+  <link name="$(arg robot_name)_base_link">
     <visual>
       <origin xyz="0 0 0.0" rpy="0 0 0"/>
@@ -30,11 +30,11 @@
   </link>
   <!-- base joint -->
-  <joint name="base_joint" type="fixed">
-    <parent link="base_footprint"/>
-    <child link="base_link"/>
+  <joint name="$(arg robot_name)_base_joint" type="fixed">
+    <parent link="$(arg robot_name)_base_footprint"/>
+    <child link="$(arg robot_name)_base_link"/>
     <origin xyz="0.0 0.0 0.076" rpy="0 0 0"/>
   </joint>
   <!-- laser link -->
-  <link name="laser_link">
+  <link name="$(arg robot_name)_laser_link">
     <visual>
       <origin xyz="0 0 0" rpy="0 0 0"/>
@@ -61,11 +61,11 @@
   </link>
   <!-- laser joint -->
-  <joint name="laser_joint" type="fixed">
-    <parent link="base_link"/>
-    <child link="laser_link"/>
+  <joint name="$(arg robot_name)_laser_joint" type="fixed">
+    <parent link="$(arg robot_name)_base_link"/>
+    <child link="$(arg robot_name)_laser_link"/>
     <origin xyz="0 0 0.075"/>
   </joint>
   <!-- imu link -->
-  <link name="imu_link">
+  <link name="$(arg robot_name)_imu_link">
     <visual>
       <origin xyz="0 0 0.0" rpy="0 0 0"/>
@@ -86,11 +86,11 @@
   </link>
   <!-- imu joint -->
-  <joint name="imu_joint" type="fixed">
-    <parent link="base_link"/>
-    <child link="imu_link"/>
+  <joint name="$(arg robot_name)_imu_joint" type="fixed">
+    <parent link="$(arg robot_name)_base_link"/>
+    <child link="$(arg robot_name)_imu_link"/>
     <origin xyz="0 0 0.02"/>
   </joint>
   <!-- left_wheel link -->
-  <link name="left_wheel_link">
+  <link name="$(arg robot_name)_left_wheel_link">
     <visual>
       <origin xyz="0 0 0" rpy="1.57079 0 0"/>
@@ -117,12 +117,12 @@
   </link>
   <!-- left_wheel joint -->
-  <joint name="left_wheel_joint" type="continuous">
-    <parent link="base_link"/>
-    <child link="left_wheel_link"/>
+  <joint name="$(arg robot_name)_left_wheel_joint" type="continuous">
+    <parent link="$(arg robot_name)_base_link"/>
+    <child link="$(arg robot_name)_left_wheel_link"/>
     <origin xyz="-0.02 0.10 -0.06"/>
     <axis xyz="0 1 0"/>
   </joint>
   <!-- right_wheel link -->
-  <link name="right_wheel_link">
+  <link name="$(arg robot_name)_right_wheel_link">
     <visual>
       <origin xyz="0 0 0" rpy="1.57079 0 0"/>
@@ -149,12 +149,12 @@
   </link>
   <!-- right_wheel joint -->
-  <joint name="right_wheel_joint" type="continuous">
-    <parent link="base_link"/>
-    <child link="right_wheel_link"/>
+  <joint name="$(arg robot_name)_right_wheel_joint" type="continuous">
+    <parent link="$(arg robot_name)_base_link"/>
+    <child link="$(arg robot_name)_right_wheel_link"/>
     <origin xyz="-0.02 -0.10 -0.06"/>
     <axis xyz="0 1 0"/>
   </joint>
   <!-- fornt caster link -->
-  <link name="front_caster_link">
+  <link name="$(arg robot_name)_front_caster_link">
     <visual>
       <origin xyz="0 0 0" rpy="1.57079 0 0"/>
@@ -181,14 +181,14 @@
   </link>
   <!-- front caster joint -->
-  <joint name="front_caster_joint" type="fixed">
-    <parent link="base_link"/>
-    <child link="front_caster_link"/>
+  <joint name="$(arg robot_name)_front_caster_joint" type="fixed">
+    <parent link="$(arg robot_name)_base_link"/>
+    <child link="$(arg robot_name)_front_caster_link"/>
     <origin xyz="0.06 0.0 -0.076"/>
     <axis xyz="0 1 0"/>
   </joint>
-  <gazebo reference="front_caster_link">
+  <gazebo reference="$(arg robot_name)_front_caster_link">
     <material>Gazebo/Black</material>
   </gazebo>
-  <gazebo reference="front_caster_link">
+  <gazebo reference="$(arg robot_name)_front_caster_link">
     <mu1 value="0.0"/>
     <mu2 value="0.0"/>
@@ -197,5 +197,5 @@
   </gazebo>
   <!-- after caster link -->
-  <link name="after_caster_link">
+  <link name="$(arg robot_name)_after_caster_link">
     <visual>
       <origin xyz="0 0 0" rpy="1.57079 0 0"/>
@@ -222,14 +222,14 @@
   </link>
   <!-- after caster joint -->
-  <joint name="after_caster_joint" type="fixed">
-    <parent link="base_link"/>
-    <child link="after_caster_link"/>
+  <joint name="$(arg robot_name)_after_caster_joint" type="fixed">
+    <parent link="$(arg robot_name)_base_link"/>
+    <child link="$(arg robot_name)_after_caster_link"/>
     <origin xyz="-0.06 0.0 -0.076"/>
     <axis xyz="0 1 0"/>
   </joint>
-  <gazebo reference="after_caster_link">
+  <gazebo reference="$(arg robot_name)_after_caster_link">
     <material>Gazebo/Black</material>
   </gazebo>
-  <gazebo reference="after_caster_link">
+  <gazebo reference="$(arg robot_name)_after_caster_link">
     <mu1 value="0.0"/>
     <mu2 value="0.0"/>
@@ -246,6 +246,6 @@
       <update_rate>30</update_rate>
       <!-- wheels -->
-      <left_joint>left_wheel_joint</left_joint>
-      <right_joint>right_wheel_joint</right_joint>
+      <left_joint>$(arg robot_name)_left_wheel_joint</left_joint>
+      <right_joint>$(arg robot_name)_right_wheel_joint</right_joint>
       <!-- kinematics -->
       <wheel_separation>0.2</wheel_separation>
@@ -258,10 +258,10 @@
       <publish_odom_tf>true</publish_odom_tf>
       <publish_wheel_tf>false</publish_wheel_tf>
-      <odometry_frame>odom</odometry_frame>
-      <robot_base_frame>base_footprint</robot_base_frame>
+      <odometry_frame>$(arg robot_name)_odom</odometry_frame>
+      <robot_base_frame>$(arg robot_name)_base_footprint</robot_base_frame>
     </plugin>
   </gazebo>
-  <gazebo reference="imu_link">
-    <sensor name="imu_sensor" type="imu">
+  <gazebo reference="$(arg robot_name)_imu_link">
+    <sensor name="$(arg robot_name)_imu_sensor" type="imu">
       <plugin filename="libgazebo_ros_imu_sensor.so" name="imu_plugin">
         <ros>
@@ -330,6 +330,6 @@
     </sensor>
   </gazebo>
-  <gazebo reference="laser_link">
-    <sensor name="laser_sensor" type="ray">
+  <gazebo reference="$(arg robot_name)_laser_link">
+    <sensor name="$(arg robot_name)_laser_sensor" type="ray">
       <always_on>true</always_on>
       <visualize>true</visualize>
@@ -356,5 +356,5 @@
         </noise>
       </ray>
-      <plugin name="laserscan" filename="libgazebo_ros_ray_sensor.so">
+      <plugin name="$(arg robot_name)_laserscan" filename="libgazebo_ros_ray_sensor.so">
         <ros>
           <namespace>/$(arg robot_name)</namespace>
@@ -362,5 +362,5 @@
         </ros>
         <output_type>sensor_msgs/LaserScan</output_type>
-        <frame_name>laser_link</frame_name>
+        <frame_name>$(arg robot_name)_laser_link</frame_name>
       </plugin>
     </sensor>
